Commit message: Add files via upload

File: urdf/my_robotic_arm.urdf (robot description, URDF)
Before this commit: robot simple_three_dof_robotic_arm, 5 links, 4 joints
Links:
- added link button1, mass 0.1; collision box size=0.1 0.1 0.1; visual box size=0.1 0.1 0.1
- added link button2, mass 0.1; collision box size=0.1 0.1 0.1; visual box size=0.1 0.1 0.1
- added link button3, mass 0.1; collision box size=0.1 0.1 0.1; visual box size=0.1 0.1 0.1
- added link button4, mass 0.1; collision box size=0.1 0.1 0.1; visual box size=0.1 0.1 0.1
- added link button5, mass 0.1; collision box size=0.1 0.1 0.1; visual box size=0.1 0.1 0.1
- added link dummy_link
- link base_link: mass 10.0 -> 0.1
- link extendable_part: geometry collision cylinder length=0.2 radius=0.05; visual cylinder length=0.5 radius=0.01
Joints:
- added joint button1_joint: type fixed, parent base_link, child button1, origin xyz=0.9 0 0.1 rpy=0 0 0
- added joint button2_joint: type fixed, parent base_link, child button2, origin xyz=0.9 0 0.3 rpy=0 0 0
- added joint button3_joint: type fixed, parent base_link, child button3, origin xyz=0.9 0 0.5 rpy=0 0 0
- added joint button4_joint: type fixed, parent base_link, child button4, origin xyz=0.9 0 0.7 rpy=0 0 0
- added joint button5_joint: type fixed, parent base_link, child button5, origin xyz=0.9 0 0.9 rpy=0 0 0
- added joint dummy_joint: type fixed, parent dummy_link, child base_link, origin xyz=0 0 0 rpy=0 0 0
- joint joint1: limit lower=-1.5708 upper=1.5708 effort=10 velocity=1.0 -> lower=-1.5708 upper=2.09 effort=10 velocity=1.0
- joint joint2: limit lower=-1.5708 upper=1.5708 effort=10 velocity=1.0 -> lower=-1.5708 upper=2.09 effort=10 velocity=1.0
- joint prismatic_joint: limit lower=0 upper=0.15 effort=5 velocity=0.02 -> lower=0 upper=0.3 effort=5 velocity=6.0; origin xyz=0 0 0.15 rpy=0 0 0 -> xyz=0 0 0.1 rpy=0 0 0
